File: hardware/lipo-booster.sch (EAGLE design)
At the start: 33 parts, among them IC1 MCP73833-UN, J2 USB, Q1 BSS84, Q2 BSS84, U1 TEXAS_INSTRUMENTS_TPS61032PWP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

Commit message: Updated design with pcb layout suggestions from reddit thread
Parts:
- LED4: value PWR_ON -> ON
Changed lines of the file:
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@@
 </classes>
 <parts>
-<part name="LOGO1" library="SparkFun-Aesthetics" deviceset="OSHW-LOGO" device="S"/>
-<part name="FRAME2" library="SparkFun-Aesthetics" deviceset="FRAME-A4L" device=""/>
-<part name="J1" library="SparkFun-Connectors" deviceset="CONN_08" device="&quot;"/>
+<part name="LOGO1" library="SparkFun-Aesthetics" library_urn="urn:adsk.eagle:library:507" deviceset="OSHW-LOGO" device="S" package3d_urn="urn:adsk.eagle:package:37099/1"/>
+<part name="FRAME2" library="SparkFun-Aesthetics" library_urn="urn:adsk.eagle:library:507" deviceset="FRAME-A4L" device=""/>
+<part name="J1" library="SparkFun-Connectors" library_urn="urn:adsk.eagle:library:513" deviceset="CONN_08" device="&quot;" package3d_urn="urn:adsk.eagle:package:38138/1"/>
 <part name="U$1" library="microbuilder" deviceset="GND" device=""/>
 <part name="U$21" library="microbuilder" deviceset="GND" device=""/>
@@
 <part name="C5" library="resistor" library_urn="urn:adsk.eagle:library:348" deviceset="C-EU" device="C0603" package3d_urn="urn:adsk.eagle:package:23616/2" value="2.2uF"/>
 <part name="C6" library="resistor" library_urn="urn:adsk.eagle:library:348" deviceset="CPOL-EU" device="CT3528" package3d_urn="urn:adsk.eagle:package:23325/2" value="220uF"/>
-<part name="LED4" library="led" library_urn="urn:adsk.eagle:library:259" deviceset="LED" device="CHIP-LED0603" package3d_urn="urn:adsk.eagle:package:15819/3" value="PWR_ON"/>
+<part name="LED4" library="led" library_urn="urn:adsk.eagle:library:259" deviceset="LED" device="CHIP-LED0603" package3d_urn="urn:adsk.eagle:package:15819/3" value="ON"/>
 <part name="GND14" library="supply1" library_urn="urn:adsk.eagle:library:371" deviceset="GND" device=""/>
 <part name="R11" library="resistor" deviceset="R-EU_" device="R0603" value="470"/>
@@
 </part>
 <part name="P+3" library="supply1" library_urn="urn:adsk.eagle:library:371" deviceset="+5V" device=""/>
-<part name="Q2" library="transistor-small-signal" library_urn="urn:adsk.eagle:library:401" deviceset="BSS84" device="" package3d_urn="urn:adsk.eagle:package:29752/1"/>
-<part name="Q1" library="transistor-small-signal" library_urn="urn:adsk.eagle:library:401" deviceset="BSS84" device="" package3d_urn="urn:adsk.eagle:package:29752/1"/>
+<part name="Q2" library="transistor-small-signal" library_urn="urn:adsk.eagle:library:401" deviceset="BSS84" device="" package3d_urn="urn:adsk.eagle:package:28738/2"/>
+<part name="Q1" library="transistor-small-signal" library_urn="urn:adsk.eagle:library:401" deviceset="BSS84" device="" package3d_urn="urn:adsk.eagle:package:28738/2"/>
 <part name="J2" library="audio amplifier example" library_urn="urn:adsk.eagle:library:970892" deviceset="1981584-1" device="" package3d_urn="urn:adsk.eagle:package:970926/2" value="USB"/>
 <part name="J3" library="adafruit" library_urn="urn:adsk.eagle:library:420" deviceset="JST_2PIN" device="-THM" package3d_urn="urn:adsk.eagle:package:6240693/1"/>

Commit message: Small change to schematic to change transistor and update of photo
Parts:
- removed Q1: BSS84, transistor-small-signal:BSS84
- added Q3: MMUN2133LT1G, transistor-pnp:MUN2114T1
Connections:
- net +5V: now also Q3.E; no longer Q1.S
- net N$32: now also Q3.B; no longer Q1.G
- net PWR_LBO: now also Q3.C; no longer Q1.D
Other:
- moved on the sheet: LED4, R11
Changed lines of the file:
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@@
 <part name="P+3" library="supply1" library_urn="urn:adsk.eagle:library:371" deviceset="+5V" device=""/>
 <part name="Q2" library="transistor-small-signal" library_urn="urn:adsk.eagle:library:401" deviceset="BSS84" device="" package3d_urn="urn:adsk.eagle:package:28738/2"/>
-<part name="Q1" library="transistor-small-signal" library_urn="urn:adsk.eagle:library:401" deviceset="BSS84" device="" package3d_urn="urn:adsk.eagle:package:28738/2"/>
 <part name="J2" library="audio amplifier example" library_urn="urn:adsk.eagle:library:970892" deviceset="1981584-1" device="" package3d_urn="urn:adsk.eagle:package:970926/2" value="USB"/>
 <part name="J3" library="adafruit" library_urn="urn:adsk.eagle:library:420" deviceset="JST_2PIN" device="-THM" package3d_urn="urn:adsk.eagle:package:6240693/1"/>
+<part name="Q3" library="transistor-pnp" library_urn="urn:adsk.eagle:library:399" deviceset="MUN2114*" device="" package3d_urn="urn:adsk.eagle:package:28754/2" technology="T1" value="MMUN2133LT1G"/>
 </parts>
 <sheets>
@@
 <attribute name="VALUE" x="178.943" y="41.1226" size="1.778" layer="96"/>
 </instance>
-<instance part="LED4" gate="G$1" x="218.44" y="38.1" smashed="yes">
-<attribute name="NAME" x="214.376" y="33.528" size="1.778" layer="95" rot="R90"/>
-<attribute name="VALUE" x="221.615" y="30.988" size="1.778" layer="96" rot="R90"/>
-</instance>
-<instance part="GND14" gate="1" x="218.44" y="25.4" smashed="yes">
-<attribute name="VALUE" x="215.9" y="22.86" size="1.778" layer="96"/>
-</instance>
-<instance part="R11" gate="G$1" x="218.44" y="53.34" smashed="yes" rot="R90">
-<attribute name="NAME" x="216.9414" y="49.53" size="1.778" layer="95" rot="R90"/>
-<attribute name="VALUE" x="221.742" y="49.53" size="1.778" layer="96" rot="R90"/>
-</instance>
-<instance part="P+2" gate="1" x="218.44" y="66.04" smashed="yes">
-<attribute name="VALUE" x="215.9" y="60.96" size="1.778" layer="96" rot="R90"/>
+<instance part="LED4" gate="G$1" x="223.52" y="38.1" smashed="yes">
+<attribute name="NAME" x="219.456" y="33.528" size="1.778" layer="95" rot="R90"/>
+<attribute name="VALUE" x="226.695" y="30.988" size="1.778" layer="96" rot="R90"/>
+</instance>
+<instance part="GND14" gate="1" x="223.52" y="25.4" smashed="yes">
+<attribute name="VALUE" x="220.98" y="22.86" size="1.778" layer="96"/>
+</instance>
+<instance part="R11" gate="G$1" x="223.52" y="53.34" smashed="yes" rot="R90">
+<attribute name="NAME" x="222.0214" y="49.53" size="1.778" layer="95" rot="R90"/>
+<attribute name="VALUE" x="226.822" y="49.53" size="1.778" layer="96" rot="R90"/>
+</instance>
+<instance part="P+2" gate="1" x="223.52" y="66.04" smashed="yes">
+<attribute name="VALUE" x="220.98" y="60.96" size="1.778" layer="96" rot="R90"/>
 </instance>
 <instance part="LED3" gate="G$1" x="195.58" y="33.02" smashed="yes">
@@
 <attribute name="VALUE" x="231.14" y="139.7" size="1.778" layer="96" rot="MR180"/>
 </instance>
-<instance part="Q1" gate="G$1" x="195.58" y="53.34" smashed="yes">
-<attribute name="NAME" x="198.12" y="53.34" size="1.778" layer="95"/>
-<attribute name="VALUE" x="198.12" y="50.8" size="1.778" layer="96"/>
-</instance>
 <instance part="J2" gate="G$1" x="20.32" y="121.92" smashed="yes" rot="MR0">
 <attribute name="NAME" x="25.4" y="130.81" size="2.54" layer="95" font="vector" ratio="12" rot="MR0"/>
@@
 <attribute name="NAME" x="21.59" y="104.775" size="1.778" layer="95" rot="MR0"/>
 <attribute name="VALUE" x="21.59" y="93.98" size="1.778" layer="96" rot="MR0"/>
+</instance>
+<instance part="Q3" gate="G$1" x="193.04" y="53.34" smashed="yes">
+<attribute name="NAME" x="198.12" y="55.88" size="1.778" layer="95"/>
+<attribute name="VALUE" x="198.12" y="53.34" size="1.778" layer="96"/>
 </instance>
 </instances>
@@
 <pinref part="GND14" gate="1" pin="GND"/>
 <pinref part="LED4" gate="G$1" pin="C"/>
-<wire x1="218.44" y1="27.94" x2="218.44" y2="33.02" width="0.1524" layer="91"/>
+<wire x1="223.52" y1="27.94" x2="223.52" y2="33.02" width="0.1524" layer="91"/>
 </segment>
 <segment>
@@
 <wire x1="195.58" y1="58.42" x2="195.58" y2="60.96" width="0.1524" layer="91"/>
 <junction x="195.58" y="60.96"/>
-<pinref part="Q1" gate="G$1" pin="S"/>
+<pinref part="Q3" gate="G$1" pin="E"/>
 </segment>
 <segment>
 <pinref part="P+2" gate="1" pin="+5V"/>
 <pinref part="R11" gate="G$1" pin="2"/>
-<wire x1="218.44" y1="63.5" x2="218.44" y2="58.42" width="0.1524" layer="91"/>
+<wire x1="223.52" y1="63.5" x2="223.52" y2="58.42" width="0.1524" layer="91"/>
 </segment>
 <segment>
@@
 <junction x="195.58" y="45.72"/>
 <label x="198.12" y="45.72" size="1.778" layer="95"/>
-<pinref part="Q1" gate="G$1" pin="D"/>
+<pinref part="Q3" gate="G$1" pin="C"/>
 </segment>
 </net>
@@
 <wire x1="142.24" y1="45.72" x2="149.86" y2="45.72" width="0.1524" layer="91"/>
 <wire x1="149.86" y1="45.72" x2="149.86" y2="38.1" width="0.1524" layer="91"/>
-<wire x1="149.86" y1="38.1" x2="187.96" y2="38.1" width="0.1524" layer="91"/>
-<wire x1="187.96" y1="38.1" x2="187.96" y2="55.88" width="0.1524" layer="91"/>
-<wire x1="187.96" y1="55.88" x2="190.5" y2="55.88" width="0.1524" layer="91"/>
-<pinref part="Q1" gate="G$1" pin="G"/>
+<wire x1="149.86" y1="38.1" x2="185.42" y2="38.1" width="0.1524" layer="91"/>
+<wire x1="185.42" y1="38.1" x2="185.42" y2="53.34" width="0.1524" layer="91"/>
+<pinref part="Q3" gate="G$1" pin="B"/>
 </segment>
 </net>
@@
 <pinref part="R11" gate="G$1" pin="1"/>
 <pinref part="LED4" gate="G$1" pin="A"/>
-<wire x1="218.44" y1="48.26" x2="218.44" y2="40.64" width="0.1524" layer="91"/>
-</segment>
-</net>
+<wire x1="223.52" y1="48.26" x2="223.52" y2="40.64" width="0.1524" layer="91"/>
+</segment>
+</net>
